Commit message: fix honeybadger.urdf

File: unitree_robots/honeybadger/urdf/honeybadger.urdf (robot description, URDF)
Before this commit: robot honeybadger, 17 links, 16 joints
Joints:
- joint FL_calf_joint: limit (none) -> lower=-3.14 upper=3.14 effort=0 velocity=0
- joint FL_hip_joint: limit (none) -> lower=-3.14 upper=3.14 effort=0 velocity=0
- joint FL_thigh_joint: limit (none) -> lower=-3.14 upper=3.14 effort=0 velocity=0
- joint FR_calf_joint: limit (none) -> lower=-3.14 upper=3.14 effort=0 velocity=0
- joint FR_hip_joint: limit (none) -> lower=-3.14 upper=3.14 effort=0 velocity=0
- joint FR_thigh_joint: limit (none) -> lower=-3.14 upper=3.14 effort=0 velocity=0
- joint RL_calf_joint: limit (none) -> lower=-3.14 upper=3.14 effort=0 velocity=0
- joint RL_hip_joint: limit (none) -> lower=-3.14 upper=3.14 effort=0 velocity=0
- joint RL_thigh_joint: limit (none) -> lower=-3.14 upper=3.14 effort=0 velocity=0
- joint RR_calf_joint: limit (none) -> lower=-3.14 upper=3.14 effort=0 velocity=0
- joint RR_hip_joint: limit (none) -> lower=-3.14 upper=3.14 effort=0 velocity=0
- joint RR_thigh_joint: limit (none) -> lower=-3.14 upper=3.14 effort=0 velocity=0
- joint front_body_joint: axis 0 0 -1 -> 0 0 1; limit (none) -> lower=-3.14 upper=3.14 effort=0 velocity=0
- joint head_joint: axis 0.368847929175079 0 -0.929489755265358 -> 0 0 -1; limit (none) -> lower=-3.14 upper=3.14 effort=0 velocity=0
- joint neck_joint: limit (none) -> lower=-3.14 upper=3.14 effort=0 velocity=0
- joint rear_body_joint: limit (none) -> lower=-3.14 upper=3.14 effort=0 velocity=0
