Commit message: add big red dog uie

File: unitree_robots/g7_plus/urdf/g7_plus.urdf (robot description, URDF)
Before this commit: robot g7_plus, 12 links, 11 joints
Joints:
- joint FL_wheel_joint: limit lower=-3.14159 upper=3.14159 effort=20 velocity=10 -> (none); type revolute -> continuous
- joint FR_wheel_joint: limit lower=-3.14159 upper=3.14159 effort=20 velocity=10 -> (none); type revolute -> continuous
- joint RL_wheel_joint: limit lower=-3.14159 upper=3.14159 effort=20 velocity=10 -> (none); type revolute -> continuous
- joint RR_wheel_joint: limit lower=-3.14159 upper=3.14159 effort=20 velocity=10 -> (none); type revolute -> continuous
