Commit message: add big red dig cpc arm and fix big red dog uie urdf

File: unitree_robots/bigreddog_cpc_arm/urdf/bigreddog_cpc_arm.urdf (robot description, URDF)
Before this commit: robot bigreddog_uie, 17 links, 16 joints
Links:
- added link S0_base_link, mass 0.50000000; collision cylinder length=0.04 radius=0.045; visual mesh filename=../meshes/S0_base_link.STL
- added link S0_f1_link, mass 0.00100000; collision box size=0.00782 0.039 0.01; visual mesh filename=../meshes/S0_f1_link.STL
- added link S0_f2_link, mass 0.00100000; collision box size=0.00782 0.039 0.01; visual mesh filename=../meshes/S0_f2_link.STL
- added link S0_link1, mass 0.50000000; collision cylinder length=0.09 radius=0.03; visual mesh filename=../meshes/S0_link1.STL
- added link S0_link2, mass 0.50000000; collision cylinder length=0.08 radius=0.0224; collision cylinder length=0.09 radius=0.03
- added link S0_link3, mass 0.50000000; collision cylinder length=0.015 radius=0.0225; collision cylinder length=0.085 radius=0.025
- added link S0_link4, mass 0.50000000; collision cylinder length=0.084 radius=0.023; visual mesh filename=../meshes/S0_link4.STL
- added link S0_link5, mass 0.50000000; collision cylinder length=0.086 radius=0.023; visual mesh filename=../meshes/S0_link5.STL
- added link S0_link6, mass 0.50000000; collision box size=0.026 0.072 0.018; collision cylinder length=0.012 radius=0.023
Joints:
- added joint S0_base_joint: type fixed, parent base_link, child S0_base_link, origin xyz=0 0.000216697742987104 0.0625 rpy=0 0 0, axis 0 0 0
- added joint S0_f1_joint: type fixed, parent S0_link6, child S0_f1_link, origin xyz=0.0129725087784923 -0.0887995988812726 -0.000303439432622427 rpy=0 0 0, axis 0 0 0
- added joint S0_f2_joint: type fixed, parent S0_link6, child S0_f2_link, origin xyz=-0.0120533576268614 -0.0888345486713001 0.000382133817736496 rpy=0 0 0, axis 0 0 0
- added joint S0_link1_joint: type revolute, parent S0_base_link, child S0_link1, origin xyz=0 0 0.049 rpy=0 0 0, axis 0 0 1, limit lower=-6.283185307179586 upper=6.283185307179586 effort=28.0 velocity=3.141592653589793
- added joint S0_link2_joint: type revolute, parent S0_link1, child S0_link2, origin xyz=-0.000305444697530935 -0.0390379384646319 0.045 rpy=0 0 0, axis 0 1 0, limit lower=-6.283185307179586 upper=6.283185307179586 effort=28.0 velocity=3.141592653589793
- added joint S0_link3_joint: type revolute, parent S0_link2, child S0_link3, origin xyz=-0.185297118289125 0.000607376944143097 0.00087579391463799 rpy=0 0 0, axis 0 1 0, limit lower=-6.283185307179586 upper=6.283185307179586 effort=28.0 velocity=3.141592653589793
- added joint S0_link4_joint: type revolute, parent S0_link3, child S0_link4, origin xyz=-0.108475817681094 0.082686442944425 -0.00111853667411776 rpy=0 0 0, axis 0 1 0, limit lower=-6.283185307179586 upper=6.283185307179586 effort=28.0 velocity=3.141592653589793
- added joint S0_link5_joint: type revolute, parent S0_link4, child S0_link5, origin xyz=-9.13167272780235E-05 0.0236071132698339 0.0487120070783628 rpy=0 0 0, axis 0 0 1, limit lower=-6.283185307179586 upper=6.283185307179586 effort=28.0 velocity=3.141592653589793
- added joint S0_link6_joint: type revolute, parent S0_link5, child S0_link6, origin xyz=-8.44278083899641E-05 -0.0522843493873027 0.028030887034242 rpy=0 0 0, axis 0 1 0, limit lower=-6.283185307179586 upper=6.283185307179586 effort=28.0 velocity=3.141592653589793
