Commit message: fix big reddog cpc arm urdf

File: unitree_robots/bigreddog/urdf/big_reddog_arm.urdf (robot description, URDF)
Before this commit: robot big_reddog, 44 links, 43 joints
Links:
- added link S0_ee_link, mass 0.001
- link S0_base_link: geometry collision cylinder length=0.04 radius=0.045; visual mesh filename=../meshes/S0_base_link.STL
- link S0_f1_link: geometry collision box size=0.00782 0.039 0.01; visual mesh filename=../meshes/S0_f1_link.STL
- link S0_f2_link: geometry collision box size=0.00782 0.039 0.01; visual mesh filename=../meshes/S0_f2_link.STL
- link S0_link1: geometry collision cylinder length=0.09 radius=0.03; visual mesh filename=../meshes/S0_link1.STL
- link S0_link2: geometry collision cylinder length=0.08 radius=0.0224; collision cylinder length=0.09 radius=0.03
- link S0_link3: geometry collision cylinder length=0.015 radius=0.0225; collision cylinder length=0.085 radius=0.025
- link S0_link4: geometry collision cylinder length=0.084 radius=0.023; visual mesh filename=../meshes/S0_link4.STL
- link S0_link5: geometry collision cylinder length=0.086 radius=0.023; visual mesh filename=../meshes/S0_link5.STL
- link S0_link6: geometry collision box size=0.026 0.072 0.018; collision cylinder length=0.012 radius=0.023
Joints:
- removed joint S0_base_link_joint
- added joint S0_base_joint: type fixed, parent base_link, child S0_base_link, origin xyz=0 0.000216697742987104 0.0625 rpy=0 0 0, axis 0 0 0
- added joint S0_ee_joint: type fixed, parent S0_link6, child S0_ee_link, origin xyz=0 -0.1085 0 rpy=0 0 -1.5708, axis 0 0 0
- joint S0_link1_joint: limit lower=-3.14 upper=3.14 effort=147.0 velocity=6.28 -> lower=-6.283185307179586 upper=6.283185307179586 effort=28.0 velocity=3.141592653589793
- joint S0_link2_joint: limit lower=-3.14 upper=3.14 effort=147.0 velocity=6.28 -> lower=-6.283185307179586 upper=6.283185307179586 effort=28.0 velocity=3.141592653589793
- joint S0_link3_joint: limit lower=-3.14 upper=3.14 effort=147.0 velocity=6.28 -> lower=-6.283185307179586 upper=6.283185307179586 effort=28.0 velocity=3.141592653589793
- joint S0_link4_joint: limit lower=-3.14 upper=3.14 effort=147.0 velocity=6.28 -> lower=-6.283185307179586 upper=6.283185307179586 effort=28.0 velocity=3.141592653589793
- joint S0_link5_joint: limit lower=-3.14 upper=3.14 effort=147.0 velocity=6.28 -> lower=-6.283185307179586 upper=6.283185307179586 effort=28.0 velocity=3.141592653589793
- joint S0_link6_joint: limit lower=-3.14 upper=3.14 effort=147.0 velocity=6.28 -> lower=-6.283185307179586 upper=6.283185307179586 effort=28.0 velocity=3.141592653589793

File: unitree_robots/bigreddog_cpc_arm/urdf/bigreddog_cpc_arm.urdf (robot description, URDF)
Before this commit: robot bigreddog_CPC, 26 links, 25 joints
Links:
- added link S0_ee_link, mass 0.001
- link FL_calf_link: geometry collision box size=0.115 0.015 0.06; collision cylinder length=0.145 radius=0.015
- link FR_calf_link: geometry collision box size=0.115 0.015 0.06; collision cylinder length=0.145 radius=0.015
- link RL_calf_link: geometry collision box size=0.115 0.015 0.06; collision cylinder length=0.145 radius=0.015
- link RR_calf_link: geometry collision box size=0.115 0.015 0.06; collision cylinder length=0.145 radius=0.015
Joints:
- added joint S0_ee_joint: type fixed, parent S0_link6, child S0_ee_link, origin xyz=0 -0.1085 0 rpy=0 0 -1.5708, axis 0 0 0
