Commit message: fix big reddog uie urdf

File: unitree_robots/bigreddog_uie/urdf/bigreddog_uie.urdf (robot description, URDF)
Before this commit: robot bigreddog_uie, 17 links, 16 joints
Links:
- link FL_calf_link: geometry collision box size=0.115 0.015 0.06; collision cylinder length=0.145 radius=0.015
- link FR_calf_link: geometry collision box size=0.115 0.015 0.06; collision cylinder length=0.145 radius=0.015
- link RL_calf_link: geometry collision box size=0.115 0.015 0.06; collision cylinder length=0.145 radius=0.015
- link RR_calf_link: geometry collision box size=0.115 0.015 0.06; collision cylinder length=0.145 radius=0.015
