Commit message: add joint limit to bigreddog_plus urdf

File: unitree_robots/bigreddog_plus/urdf/bigreddog_plus.urdf (robot description, URDF)
Before this commit: robot bigreddog_plus, 17 links, 16 joints
Joints:
- joint FL_calf_joint: limit (none) -> lower=-2.792 upper=2.809 effort=40.0 velocity=20.
- joint FL_hip_joint: limit (none) -> lower=-1.0472 upper=1.0472 effort=40.0 velocity=20.
- joint FL_thigh_joint: limit (none) -> lower=-2.583 upper=2.286 effort=40.0 velocity=20.
- joint FR_calf_joint: limit (none) -> lower=-2.792 upper=2.809 effort=40.0 velocity=20.
- joint FR_hip_joint: limit (none) -> lower=-1.0472 upper=1.0472 effort=40.0 velocity=20.
- joint FR_thigh_joint: limit (none) -> lower=-2.583 upper=2.286 effort=40.0 velocity=20.
- joint RL_calf_joint: limit (none) -> lower=-2.792 upper=2.809 effort=80.0 velocity=20.
- joint RL_hip_joint: limit (none) -> lower=-1.0472 upper=1.0472 effort=40.0 velocity=20.
- joint RL_thigh_joint: limit (none) -> lower=-2.583 upper=2.286 effort=40.0 velocity=20.
- joint RR_calf_joint: limit (none) -> lower=-2.792 upper=2.809 effort=40.0 velocity=20.
- joint RR_hip_joint: limit (none) -> lower=-1.0472 upper=1.0472 effort=40.0 velocity=20.
- joint RR_thigh_joint: limit (none) -> lower=-2.583 upper=2.286 effort=40.0 velocity=20.
